Commit message: Arreglo de camaras y uso de nube de puntos

File: description/camara_profundidad.xacro (robot description, xacro)
@@ -22,5 +22,5 @@
     <gazebo reference="camara_vinculo">
         <material>Gazebo/Red</material>
-        <sensor name="camera" type="camera"><!-- Tipo de sensor a utilizar, en este caso LASER-->
+        <sensor name="camera" type="depth"><!-- Tipo de sensor a utilizar, en este caso LASER-->
             <pose> 0 0 0 0 0 0 </pose><!-- Punto de referencia para el sensor-->
             <visualize>true</visualize><!-- Visualizacion dentro del entorno-->
@@ -29,5 +29,5 @@
                 <horizontal_fov>1.089</horizontal_fov><!--Se estipula el ancho (o angulo de vision) de la camara en radianes-->
                 <image>
-                    <format>R8G8B8</format><!-- Sistema RGB de 8 bits-->
+                    <format>B8G8R8</format><!-- Sistema BGR de 8 bits, cambio de sistema por la camara de profundidad-->
                     <width>640</width><!-- Amcho y largo de la visualizacion de la camara-->
                     <height>480</height>
@@ -40,4 +40,7 @@
             <plugin name="camara_controller" filename="libgazebo_ros_camera.so"><!-- Controladores estandar de ROS para la visualizacion en GAZEBO-->
                 <frame_name>camara_optical_vinculo</frame_name>
+                <!-- Ingreso de límites para poder visualizar la cámara dentro de rviz2-->
+                <min_depth>0.1</min_depth>
+                <max_depth>100.0</max_depth>
             </plugin>
         </sensor>

File: description/lidar.xacro (robot description, xacro)
@@ -11,5 +11,5 @@
                 <box size="0.05 0.05 0.02"/>
             </geometry>
-            <material name="black"/>
+            <material name="red"/>
         </visual>
         <collision>
@@ -43,5 +43,5 @@
             <plugin name="laser_controller" filename="libgazebo_ros_ray_sensor.so"><!-- Controladores estandar de ROS para la visualizacion en GAZEBO-->
                 <ros>
-                    <argument>~/out:=scan</argument><!-- Argumento para lanzamiento del archivo dentro de ROS-->
+                    <argument>--ros-args --remap ~/out:=scan</argument><!-- Argumento para lanzamiento del archivo dentro de ROS-->
                 </ros>
                 <output_type>sensor_msgs/LaserScan</output_type><!-- Tipo de mensaje de salida-->

File: description/robot.urdf.xacro (robot description, xacro)
@@ -6,4 +6,5 @@
     <xacro:include filename="gazebo_control.xacro" />
     <xacro:include filename="lidar.xacro" />
-    <xacro:include filename="camara.xacro" />
+    <!-- <xacro:include filename="camara.xacro" /> -->
+    <xacro:include filename="camara_profundidad.xacro" />
 </robot>

File: description/robot_core.xacro (robot description, xacro)
@@ -17,4 +17,7 @@
     <material name="black">
         <color rgba="0 0 0 1"/>
+    </material>
+    <material name="red">
+        <color rgba="1 0 0 1"/>
     </material>
     <!-- CUERPO DEL ROBOT-->
